Commit message: fix urdf parsing at launch, launch in bringup

File: catkin_ws/src/auv_description/urdf/auv.urdf (robot description, URDF)
Before this commit: robot auv, 2 links, 0 joints
Links:
- removed link base_link
- removed link world
- added link auv_base; collision cylinder length=0.6 radius=0.2; visual cylinder length=0.6 radius=0.2
